Commit message: Updates to robot model file.

File: urdf/mecanum.xacro (robot description, xacro)
@@ -3,10 +3,17 @@
   <!-- include gazebo plugins -->
   <xacro:include filename="$(find mecanum_sim)/urdf/mecanum.gazebo" />
-<!--~~~~~~~~~~~~~~~~~~~~~~~~~~~~~~~~~~~~~~~~~~~~~~~~~~~~~~~~~~~~~~~~~~~~~~-->
-<!--                           LINKS                                      -->
-<!--          "distinct parts of the thing that you're making"            -->
-<!--~~~~~~~~~~~~~~~~~~~~~~~~~~~~~~~~~~~~~~~~~~~~~~~~~~~~~~~~~~~~~~~~~~~~~~-->
+  <xacro:property name="base_width" value="0.3683" />   <!-- 14.5 in -->
+  <xacro:property name="base_length" value="0.5461" />  <!-- 21.5 in -->
+  <xacro:property name="base_height" value="0.0635" />   <!-- 2.5 in  -->
+  <xacro:property name="wheel_radius" value="0.1016" /> <!-- 4.0 in  -->
+  <xacro:property name="wheel_width" value="0.0762" />  <!-- 3.0 in  -->
+  <xacro:property name="wheel_gap" value="0.0508" />    <!-- 2.0 in  -->
+  <xacro:property name="wheel_setback" value="0.041275" />    <!-- 1 5/8 in  -->
+  <xacro:property name="lidar_width" value="0.0508" />    <!-- 2.0 in  -->
+  <xacro:property name="lidar_length" value="0.0508" />    <!-- 2.0 in  -->
+  <xacro:property name="lidar_height" value="0.0762" />    <!-- 3.0 in  -->
+  <xacro:property name="lidar_setback" value="0.0127" />    <!-- 0.5 in  -->
   <!--~~~~~~~~~~~~~~~~~~~~~~~~ ~ ROBOT BASE ~ ~~~~~~~~~~~~~~~~~~~~~~~~~~~~~~-->
-  <!-- Make a box for robot base thingie -->
+  <!-- Make a box for robot base -->
   <link name="base_link">
   	<!-- Draw imaginary box around the robot for collision detection -->
@@ -14,12 +21,12 @@
       <origin xyz="0 0 0.0" rpy="0 0 0"/>
       <geometry>
-       <box size="0.6 0.5 0.1"/>
+       <box size="${base_length} ${base_width} ${base_height}"/>
       </geometry>
     </collision>
     <!-- Describe how to draw the box in 3d -->
     <visual>
-      <origin xyz="0 0 0.1" rpy="0 0 0"/>
+      <origin xyz="0 0 0.0" rpy="0 0 0"/>
       <geometry>
-	<box size="0.6 0.5 0.1"/>
+	       <box size="${base_length} ${base_width} ${base_height}"/>
       </geometry>
       <material name="red"/>
@@ -34,5 +41,5 @@
       <visual>
         <geometry>
-          <cylinder length="0.05" radius="0.1"/>
+          <cylinder length="${wheel_width}" radius="${wheel_radius}"/>
         </geometry>
         <origin rpy="${pi/2} 0 0" xyz="0 0 0"/>
@@ -40,5 +47,5 @@
       <collision>
         <geometry>
-          <cylinder length="0.05" radius="0.1"/>
+          <cylinder length="${wheel_width}" radius="${wheel_radius}"/>
         </geometry>
         <origin rpy="${pi/2} 0 0" xyz="0 0 0"/>
@@ -53,5 +60,5 @@
         <visual>
           <geometry>
-            <cylinder length="0.05" radius="0.1"/>
+            <cylinder length="${wheel_width}" radius="${wheel_radius}"/>
           </geometry>
           <origin rpy="${pi/2} 0 0" xyz="0 0 0"/>
@@ -59,5 +66,5 @@
         <collision>
           <geometry>
-            <cylinder length="0.05" radius="0.1"/>
+            <cylinder length="${wheel_width}" radius="${wheel_radius}"/>
           </geometry>
           <origin rpy="${pi/2} 0 0" xyz="0 0 0"/>
@@ -72,5 +79,5 @@
           <visual>
             <geometry>
-              <cylinder length="0.05" radius="0.1"/>
+              <cylinder length="${wheel_width}" radius="${wheel_radius}"/>
             </geometry>
             <origin rpy="${pi/2} 0 0" xyz="0 0 0"/>
@@ -78,5 +85,5 @@
           <collision>
             <geometry>
-              <cylinder length="0.05" radius="0.1"/>
+              <cylinder length="${wheel_width}" radius="${wheel_radius}"/>
             </geometry>
             <origin rpy="${pi/2} 0 0" xyz="0 0 0"/>
@@ -91,5 +98,5 @@
             <visual>
               <geometry>
-                <cylinder length="0.05" radius="0.1"/>
+                <cylinder length="${wheel_width}" radius="${wheel_radius}"/>
               </geometry>
               <origin rpy="${pi/2} 0 0" xyz="0 0 0"/>
@@ -97,5 +104,5 @@
             <collision>
               <geometry>
-                <cylinder length="0.05" radius="0.1"/>
+                <cylinder length="${wheel_width}" radius="${wheel_radius}"/>
               </geometry>
               <origin rpy="${pi/2} 0 0" xyz="0 0 0"/>
@@ -112,5 +119,5 @@
       <origin xyz="0 0 0" rpy="0 0 0"/>
       <geometry>
-       <box size="0.05 0.05 0.04"/>
+       <box size="${lidar_length} ${lidar_width} ${lidar_height}"/>
       </geometry>
     </collision>
@@ -118,5 +125,5 @@
       <origin xyz="0 0 0" rpy="0 0 0"/>
       <geometry>
-	       <box size="0.05 0.05 0.04"/>
+	       <box size="${lidar_length} ${lidar_width} ${lidar_height}"/>
       </geometry>
       <material name="red"/>
@@ -128,13 +135,8 @@
     </inertial>
   </link>
-<!--~~~~~~~~~~~~~~~~~~~~~~~~~~~~~~~~~~~~~~~~~~~~~~~~~~~~~~~~~~~~~~~~~~~~~~-->
-<!--                           JOINTS                                     -->
-<!--            "connections between the distinct parts"                  -->
-<!--~~~~~~~~~~~~~~~~~~~~~~~~~~~~~~~~~~~~~~~~~~~~~~~~~~~~~~~~~~~~~~~~~~~~~~-->
-  <!-- Connect the robot to the forward facing camera -->
   <joint name="joint1" type="fixed">      <!-- Fused connection? (using continuous tilts view)-->
     <parent link="base_link"/>            <!--      robot link = parent     -->
     <child link="laser_link"/>     <!-- forward camera link = child  -->
-    <origin xyz="0.25 0 0.18" rpy="0 0 0"/>   <!-- where child is relative to parent -->
+    <origin xyz="${base_length/2 - lidar_length/2 - lidar_setback} 0 ${lidar_height}" rpy="0 0 0"/>   <!-- where child is relative to parent -->
     <axis xyz="0 0 0"/>                   <!-- ...describes the axis of rotation? -->
   </joint>
@@ -142,5 +144,5 @@
       <parent link="base_link"/>
       <child link="fl_link"/>
-      <origin rpy="0 0 0" xyz="0.3 0.25 0.1"/>
+      <origin rpy="0 0 0" xyz="${base_length/2 - wheel_setback} ${base_width/2 + wheel_gap} 0.0"/>
       <axis xyz="0 0 0"/>
       <!-- <dynamics damping="1.0" friction="0.0" spring_stiffness="1" /> -->
@@ -149,5 +151,5 @@
       <parent link="base_link"/>
       <child link="fr_link"/>
-      <origin rpy="0 0 0" xyz="0.3 -0.25 0.1"/>
+      <origin rpy="0 0 0" xyz="${base_length/2 - wheel_setback} ${-base_width/2 - wheel_gap} 0.0"/>
       <axis xyz="0 0 0"/>
       <!-- <dynamics damping="1.0" friction="0.0" spring_stiffness="1" /> -->
@@ -156,5 +158,5 @@
       <parent link="base_link"/>
       <child link="bl_link"/>
-      <origin rpy="0 0 0" xyz="-0.3 0.25 0.1"/>
+      <origin rpy="0 0 0" xyz="${-base_length/2 + wheel_setback} ${base_width/2 + wheel_gap} 0.0"/>
       <axis xyz="0 0 0"/>
       <!-- <dynamics damping="1.0" friction="0.0" spring_stiffness="1" /> -->
@@ -163,5 +165,5 @@
       <parent link="base_link"/>
       <child link="br_link"/>
-      <origin rpy="0 0 0" xyz="-0.3 -0.25 0.1"/>
+      <origin rpy="0 0 0" xyz="${-base_length/2 + wheel_setback} ${-base_width/2 - wheel_gap} 0.0"/>
       <axis xyz="0 0 0"/>
       <!-- <dynamics damping="1.0" friction="0.0" spring_stiffness="1" /> -->

Commit message: More precise measurements.

File: urdf/mecanum.xacro (robot description, xacro)
@@ -4,5 +4,5 @@
   <xacro:include filename="$(find mecanum_sim)/urdf/mecanum.gazebo" />
   <xacro:property name="base_width" value="0.3683" />   <!-- 14.5 in -->
-  <xacro:property name="base_length" value="0.5461" />  <!-- 21.5 in -->
+  <xacro:property name="base_length" value="0.549275" />  <!-- 21 5/8 in -->
   <xacro:property name="base_height" value="0.0635" />   <!-- 2.5 in  -->
   <xacro:property name="wheel_radius" value="0.1016" /> <!-- 4.0 in  -->
